File: LTELink.kicad_pcb (KiCad board)
At the start: 4 copper layers, 93.3 x 65.8 mm, 96 parts, among them IC1 RTL8305NB-VC-CG, J1 DF40HC(3.0)-100DS-0.4V(51), J2 DF40HC(3.0)-100DS-0.4V(51), J3 DF40HC(3.0)-100DS-0.4V(51), J4 1759547-1, J5 USB_A, J6 Conn_01x03_Pin, J7 Micro_SD_Card_Det1, J8 USB_A, J9 USB_C_Receptacle_USB2.0_16P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

Commit message: finalized board for fabrication
Parts:
- R6: footprint Resistor_SMD:R_0402_1005Metric -> Resistor_SMD:R_0805_2012Metric_Pad1.20x1.40mm_HandSolder
- moved R6 2.89 mm to (207.7, 77.2)
Connections:
- J4 pad 53: GND -> (no net)
Routing:
- net Net-(IC1-IBREF): track 2.90 -> 5.40 mm
- net /Compute Module/RXIP0: track 26.9 -> 28.0 mm
- net /Compute Module/RXIN0: track 26.8 -> 28.0 mm
- net /Compute Module/TXON0: track 26.9 -> 28.1 mm
- net /Compute Module/TXOP0: track 26.9 -> 27.9 mm
- net GND: vias 91 -> 97
