File: ethernet.kicad_sch (KiCad schematic)
At the start: 59 parts, among them IC1 RTL8305NB-VC-CG, Y2 X322525MOB4SI

Commit message: finalized board for fabrication
Parts:
- C1, C19, C20, C21, C27, C6: LCSC Part # (none) -> C96446
- C16, C17, C18, C22, C23, C24, C25, C26, C28, C29, C30, C31, C33, C36, C38, C39, C43, C44, C45, C46, C47, C48, C7: LCSC Part # (none) -> C15525
- C41, C42: LCSC Part # (none) -> C1547
- IC1: FT Rotation Offset (none) -> -90; LCSC Part # (none) -> C42939821
- LED1: LCSC Part # (none) -> C2297
- R10, R22, R7, R8, R9: LCSC Part # (none) -> C25123
- R11, R12, R14, R19, R4: LCSC Part # (none) -> C21189
- R13: LCSC Part # (none) -> C25867
- R6: footprint Resistor_SMD:R_0402_1005Metric -> Resistor_SMD:R_0805_2012Metric_Pad1.20x1.40mm_HandSolder; LCSC Part # (none) -> C25884; now not fitted
- Y2: LCSC Part # (none) -> C9006
