File: KiCad/LTELink/LTELink.kicad_pcb (KiCad board)
At the start: 4 copper layers, 93.3 x 65.8 mm, 97 parts, among them IC1 RTL8305NB-VC-CG, J1 DF40HC(3.0)-100DS-0.4V(51), J10 Conn_01x03_Pin, J11 Conn_01x03_Pin, J12 Conn_01x03_Pin, J2 DF40HC(3.0)-100DS-0.4V(51), J3 DF40HC(3.0)-100DS-0.4V(51), J4 1759547-1, J5 USB_A, J6 Conn_01x03_Pin, J7 Micro_SD_Card_Det1, J8 USB_A, J9 USB_C_Receptacle_USB2.0_16P, U1 LM29300T-3.3, Y2 X322525MOB4SI

Commit message: Progress on V2.0 and file structure reformat
Parts:
- removed C45, C46, C47, C48: 100n, Capacitor_SMD:C_0402_1005Metric
- removed J10, J11, J12, J6: Conn_01x03_Pin, Connector_PinHeader_2.54mm:PinHeader_1x03_P2.54mm_Vertical
- removed J8: USB_A, LTELink:902131A1011D10100
- removed the J9 at (169.6, 62.2)
- removed LED1, LED2: KT-0805G, LED_SMD:LED_0805_2012Metric
- removed LED6: KT-0603W, LED_SMD:LED_0603_1608Metric
- removed REF**: JST_GH_BM04B-GHS-TBT_1x04-1MP_P1.25mm_Vertical, Connector_JST:JST_GH_BM04B-GHS-TBT_1x04-1MP_P1.25mm_Vertical
- removed REF**: Radxa_CM5, LTELink:Radxa_CM5
- removed RJ1, RJ2, RJ3, RJ4: HR913550A, LTELink:HR913550A
- added C14: 1p, Capacitor_SMD:C_0402_1005Metric, F.Cu at (162.1, 107.0)
- added C15: 1p, Capacitor_SMD:C_0402_1005Metric, F.Cu at (162.1, 100.7)
- added C32: 1p, Capacitor_SMD:C_0402_1005Metric, F.Cu at (160.7, 91.4)
- added C34: 1p, Capacitor_SMD:C_0402_1005Metric, F.Cu at (160.7, 84.5)
- added D10: LED, LED_SMD:LED_0603_1608Metric, F.Cu at (180.3, 57.4)
- added D11: LED, LED_SMD:LED_0805_2012Metric, F.Cu at (184.0, 57.6)
- added D12: LED, LED_SMD:LED_0805_2012Metric, F.Cu at (148.7, 79.0)
- added D13: LED, LED_SMD:LED_0805_2012Metric, F.Cu at (148.7, 88.5)
- added D14: LED, LED_SMD:LED_0805_2012Metric, F.Cu at (148.7, 97.9)
- added D15: LED, LED_SMD:LED_0805_2012Metric, F.Cu at (148.7, 107.5)
- added D9: LED, LED_SMD:LED_0805_2012Metric, F.Cu at (176.6, 57.6)
- added J13: Conn_01x04, Connector_JST:JST_GH_BM04B-GHS-TBT_1x04-1MP_P1.25mm_Vertical, B.Cu at (158.5, 71.0)
- added J14: Conn_01x04, Connector_JST:JST_GH_BM04B-GHS-TBT_1x04-1MP_P1.25mm_Vertical, B.Cu at (158.5, 62.0)
- added J15: Conn_01x04, Connector_JST:JST_GH_BM04B-GHS-TBT_1x04-1MP_P1.25mm_Vertical, B.Cu at (154.2, 79.0)
- added J19: Conn_01x04, Connector_JST:JST_GH_BM04B-GHS-TBT_1x04-1MP_P1.25mm_Vertical, B.Cu at (216.2, 107.3)
- added J21: Conn_01x04, Connector_JST:JST_GH_BM04B-GHS-TBT_1x04-1MP_P1.25mm_Vertical, B.Cu at (199.2, 107.3)
- added J22: Conn_01x04, Connector_JST:JST_GH_BM04B-GHS-TBT_1x04-1MP_P1.25mm_Vertical, B.Cu at (154.2, 88.5)
- added J23: Conn_01x04, Connector_JST:JST_GH_BM04B-GHS-TBT_1x04-1MP_P1.25mm_Vertical, B.Cu at (154.2, 98.0)
- added J24: Conn_01x04, Connector_JST:JST_GH_BM04B-GHS-TBT_1x04-1MP_P1.25mm_Vertical, B.Cu at (154.2, 107.5)
- added L1: 350uH, LTELink:SOP-40_L28.1-W12.2-P1.27-LS16.00-BL, F.Cu at (171.9, 97.0)
- added R20: 75, Resistor_SMD:R_0402_1005Metric, F.Cu at (162.1, 99.8)
- added R21: 75, Resistor_SMD:R_0402_1005Metric, F.Cu at (162.0, 92.8)
- added R23: 75, Resistor_SMD:R_0402_1005Metric, F.Cu at (162.0, 85.8)
- added R24: 510, Resistor_SMD:R_0402_1005Metric, F.Cu at (150.6, 106.5)
- D2, D3, D4, D5: moved to B.Cu
- J5: value USB_A -> Conn_01x03; footprint LTELink:902131A1011D10100 -> Connector_PinHeader_2.54mm:PinHeader_1x03_P2.54mm_Vertical
- J7: footprint LTELink:XKTF015N -> LTELink:TF-SMD_TF-009
- R8: value 510 -> 75
- moved R10 84.3 mm to (150.6, 87.5), turned to 180 degrees
- moved R9 77.7 mm to (150.6, 78.0), turned to 180 degrees
- moved D5 69.3 mm to (159.3, 107.5), turned to 90 degrees
- moved J5 63.5 mm to (224.2, 58.6), turned to 180 degrees
- moved D4 41.5 mm to (159.3, 98.0), turned to 90 degrees
- moved R8 35.6 mm to (162.1, 106.1), turned to 180 degrees
- moved D3 35.1 mm to (159.3, 88.5)
- moved JP1 28.7 mm to (224.4, 101.8), turned to 90 degrees
- moved R22 27.9 mm to (150.6, 97.0)
- moved D2 23.1 mm to (159.3, 79.0), turned to 90 degrees
- moved C38 20.0 mm to (182.4, 106.5), turned to 180 degrees
- moved C39 18.6 mm to (181.8, 100.3)
- moved C43 12.0 mm to (181.4, 94.2), turned to 90 degrees
- moved C44 11.6 mm to (182.4, 87.5), turned to 180 degrees
- moved J7 2.19 mm to (230.4, 78.9), turned to -90 degrees
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Connections:
- net Net-(IC1-P0LED/DIS_EEE) renamed /Ethernet/P0LED
- C38 pad 1: Net-(C38-Pad1) -> GND
- C38 pad 2: GND -> Net-(C38-Pad2)
- C39 pad 1: Net-(C39-Pad1) -> GND
- C39 pad 2: GND -> Net-(C39-Pad2)
- C43 pad 1: Net-(C43-Pad1) -> GND
- C43 pad 2: GND -> Net-(C43-Pad2)
- C44 pad 1: Net-(C44-Pad1) -> GND
- C44 pad 2: GND -> Net-(C44-Pad2)
- D2 pad 1: /Ethernet/RXIN1 -> /Ethernet/TX1-
- D2 pad 3: /Ethernet/RXIP1 -> /Ethernet/TX1+
- D2 pad 4: /Ethernet/TXON1 -> /Ethernet/RX1-
- D2 pad 6: /Ethernet/TXOP1 -> /Ethernet/RX1+
- D3 pad 1: /Ethernet/RXIN2 -> /Ethernet/TX2-
- D3 pad 3: /Ethernet/RXIP2 -> /Ethernet/TX2+
- D3 pad 4: /Ethernet/TXON2 -> /Ethernet/RX2-
- D3 pad 6: /Ethernet/TXOP2 -> /Ethernet/RX2+
- D4 pad 1: /Ethernet/RXIN3 -> /Ethernet/TX3-
- D4 pad 3: /Ethernet/RXIP3 -> /Ethernet/TX3+
- D4 pad 4: /Ethernet/TXON3 -> /Ethernet/RX3-
- D4 pad 6: /Ethernet/TXOP3 -> /Ethernet/RX3+
- D5 pad 1: /Ethernet/RXIN4 -> /Ethernet/TX4-
- D5 pad 3: /Ethernet/RXIP4 -> /Ethernet/TX4+
- D5 pad 4: /Ethernet/TXON4 -> /Ethernet/RX4+
- D5 pad 6: /Ethernet/TXOP4 -> /Ethernet/RX4-
- D8 pad 4: /USB/J8_D+ -> /USB/J8_D-
- D8 pad 6: /USB/J8_D- -> /USB/J8_D+
- FL2 pad 1: /USB/J8_D+ -> /USB/J8_D-
- FL2 pad 2: /USB/J8_D- -> /USB/J8_D+
- FL2 pad 3: /Compute Module/USB2_HOST3_D- -> /Compute Module/USB2_HOST3_D+
- FL2 pad 4: /Compute Module/USB2_HOST3_D+ -> /Compute Module/USB2_HOST3_D-
- J3 pad 97: +5V -> +3.3V
- J4 pad 11: /Compute Module/UART1_TX -> /EC25/EC25_UART_RX
- J4 pad 13: /Compute Module/UART1_RX -> /EC25/EC25_UART_TX
- J4 pad 23: /Compute Module/UART1_RTS -> /EC25/EC25_UART_CTS
- J4 pad 25: /Compute Module/UART1_CTS -> /EC25/EC25_UART_RTS
- J4 pad 53: GND -> unconnected-(J4A-NUT-Pad53)
- J4 pad S1: GND -> unconnected-(J4-PadS1)
- J5 pad 1: +5V -> GND
- J5 pad 2: /USB/J9_J5_D- -> /Compute Module/UART2_TX
- J5 pad 3: /USB/J9_J5_D+ -> /Compute Module/UART2_RX
- R10 pad 1: /Ethernet/P4LED -> /Ethernet/P2LED
- R22 pad 1: /Ethernet/P1LED -> /Ethernet/P3LED
- R8 pad 1: /Ethernet/P2LED -> Net-(L1-Pad38)
- R9 pad 1: /Ethernet/P3LED -> /Ethernet/P1LED
- Raxda pad NUT: GND -> (no net)
Routing:
- net /Ethernet/P2LED: track 34.4 -> 109.6 mm
- net /Ethernet/P3LED: track 34.3 -> 106.7 mm
- net /Ethernet/P4LED: track 40.6 -> 101.0 mm
- net /Ethernet/P1LED: track 59.3 -> 114.5 mm
- net /Compute Module/UART1_RTS: track 38.2 -> 0.00 mm, vias 1 -> 0
- net /Compute Module/UART1_CTS: track 37.0 -> 0.65 mm, vias 1 -> 0
- net /Compute Module/UART5_RX: track 32.7 -> 0.00 mm, vias 1 -> 0
- net /Compute Module/UART5_TX: track 32.4 -> 0.00 mm, vias 1 -> 0
- net /Ethernet/RXIN1: track 59.1 -> 28.9 mm
- net /Ethernet/RXIP1: track 59.0 -> 29.3 mm
- net /Compute Module/USB_OTG_ID: track 31.2 -> 8.88 mm, vias 1 -> 0
- net /Ethernet/RX2+: track 0.00 -> 21.8 mm, vias 0 -> 1
- net /Ethernet/TXON1: track 49.1 -> 28.3 mm
- net /Ethernet/TXOP1: track 48.8 -> 28.0 mm
- net /Ethernet/TX4-: track 0.00 -> 18.5 mm, vias 0 -> 1
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Other:
- board size 93.3 x 65.8 mm -> 93.3 x 58.9 mm
- board text added: "DEBUG"
- board text added: "ETH1"
- board text added: "ETH2"
- board text added: "ETH3"
- board text added: "ETH4"
- board text added: "RX+"
- board text added: "RX-"
- board text added: "TX+"
- board text added: "TX-"
- board text added: "USB1"
- board text added: "USB2"
- board text added: "V2.0"
- board text removed: "MAVLINK"
- board text removed: "UART5"
- board text removed: "V1.0"
