File: KiCad/LTELink/sd_card.kicad_sch (KiCad schematic)
At the start: 6 parts, among them J7 Micro_SD_Card_Det1

Commit message: Progress on V2.0 and file structure reformat
Parts:
- J7: footprint LTELink:XKTF015N -> LTELink:TF-SMD_TF-009
Changed lines of the file:
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@@
 			)
 		)
-		(property "Footprint" "LTELink:XKTF015N"
+		(property "Footprint" "LTELink:TF-SMD_TF-009"
 			(at 186.69 58.42 0)
 			(hide yes)
