File: KiCad/LTELink/usb.kicad_sch (KiCad schematic)
At the start: 9 parts, among them J5 USB_A, J8 USB_A, J9 USB_C_Receptacle_USB2.0_16P

Commit message: Progress on V2.0 and file structure reformat
Parts:
- removed J5, J8: USB_A, LTELink:902131A1011D10100, symbol Connector:USB_A
- added J13, J14: Conn_01x04, Connector_JST:JST_GH_BM04B-GHS-TBT_1x04-1MP_P1.25mm_Vertical, symbol Connector_Generic:Conn_01x04
Connections:
- net +5V: now also J13.1 (Pin_1), J14.1 (Pin_1)
- net GND: now also J13.4 (Pin_4), J14.4 (Pin_4)
- net J8_D+: now also D8.6 (IO4), FL2.2, J13.2 (Pin_2); no longer D8.4 (IO3), FL2.1
- net J8_D-: now also D8.4 (IO3), FL2.1, J13.3 (Pin_3); no longer D8.6 (IO4), FL2.2
- net J9_J5_D+: now also J14.2 (Pin_2)
- net J9_J5_D-: now also J14.3 (Pin_3)
- net USB_2.0_D+: now also FL2.3; no longer FL2.4
- net USB_2.0_D-: now also FL2.4; no longer FL2.3
Other:
- moved on the sheet: FL2
