File: KiCad/LTELink/LTELink.kicad_sch (KiCad schematic)
At the start: 0 parts

Commit message: Progress on V2.0 and file structure reformat
Other:
- sheet Compute Module ports: added none; removed UART1_CTS, UART1_RTS
- sheet EC25 ports: added VBUS_DET; removed none
- sheet USB ports: added none; removed VBUS_DET
- sheet uart ports: added DEBUG_RX, DEBUG_TX; removed UART3_RX, UART3_TX

Commit message: Finalize LTELink V2 for production
Other:
- added sheet pwm (pwm.kicad_sch)
- sheet Compute Module ports: added PWM11; removed none
Changed lines of the file:
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@@
+	(wire
+		(pts
+			(xy 170.18 62.23) (xy 177.8 62.23)
+		)
+		(stroke
+			(width 0)
+			(type default)
+		)
+	)
 	(wire
 		(pts
@@
 			(width 0)
 			(type default)
+		)
+	)
+	(sheet
+		(at 177.8 50.8)
+		(size 31.75 20.32)
+		(exclude_from_sim no)
+		(in_bom yes)
+		(on_board yes)
+		(dnp no)
+		(fields_autoplaced yes)
+		(stroke
+			(width 0.1524)
+			(type solid)
+		)
+		(fill
+			(color 0 0 0 0)
+		)
+		(property "Sheetname" "pwm"
+			(at 177.8 50.0884 0)
+			(show_name no)
+			(do_not_autoplace no)
+			(effects
+				(font
+					(size 1.27 1.27)
+				)
+				(justify left bottom)
+			)
+		)
+		(property "Sheetfile" "pwm.kicad_sch"
+			(at 177.8 71.7046 0)
+			(show_name no)
+			(do_not_autoplace no)
+			(effects
+				(font
+					(size 1.27 1.27)
+				)
+				(justify left top)
+			)
+		)
+		(pin "fan_pwm" input
+			(at 177.8 62.23 180)
+			(effects
+				(font
+					(size 1.27 1.27)
+				)
+				(justify left)
+			)
+		)
+		(instances
+			(project "LTELink"
+				(path "/ebd96e19-6f65-4022-a6da-be26c0716f8e"
+					(page "8")
+				)
+			)
 		)
 	)
@@
 			)
 		)
+		(pin "PWM11" input
+			(at 170.18 62.23 0)
+			(effects
+				(font
+					(size 1.27 1.27)
+				)
+				(justify right)
+			)
+		)
