File: KiCad/LTELink/_autosave-LTELink.kicad_pcb (KiCad board)
At the start: 4 copper layers, 93.3 x 58.9 mm, 107 parts, among them IC1 RTL8305NB-VC-CG, J1 DF40HC(3.0)-100DS-0.4V(51), J13 Conn_01x04, J14 Conn_01x04, J15 Conn_01x04, J19 Conn_01x04, J2 DF40HC(3.0)-100DS-0.4V(51), J21 Conn_01x04, J22 Conn_01x04, J23 Conn_01x04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

Commit message: Finalize LTELink V2 for production
Parts:
- renumbered TP2 to RX5, TP1 to TX5
Changed lines of the file:
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@@
 		(descr "SMD pad as test Point, diameter 2.0mm")
 		(tags "test point SMD pad")
-		(property "Reference" "TP2"
+		(property "Reference" "RX5"
 			(at -2.8 0 0)
 			(layer "F.SilkS")
@@
 		(descr "SMD pad as test Point, diameter 2.0mm")
 		(tags "test point SMD pad")
-		(property "Reference" "TP1"
+		(property "Reference" "TX5"
 			(at -2.7 0 0)
 			(layer "F.SilkS")
