File: KiCad/LTELink/compute_module.kicad_sch (KiCad schematic)
At the start: 4 parts, among them J1 DF40HC(3.0)-100DS-0.4V(51), J2 DF40HC(3.0)-100DS-0.4V(51), J3 DF40HC(3.0)-100DS-0.4V(51)

Commit message: Finalize LTELink V2 for production
Connections:
- net PWM11: now reaches J1.31 (GPIO12)
- no-connect marks 181 -> 180
Changed lines of the file:
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@@
-	)
-	(no_connect
-		(at 132.08 104.14)
 	)
 	(no_connect
@@
 		(effects
 			(font
+				(size 1.27 1.27)
+			)
+			(justify left)
+		)
+	)
+	(hierarchical_label "PWM11"
+		(shape input)
+		(at 132.08 104.14 0)
+		(effects
+			(font
