File: KiCad/LTELink/uart.kicad_sch (KiCad schematic)
At the start: 5 parts, among them J19 Conn_01x04, J21 Conn_01x04, J5 Conn_01x03

Commit message: Moved LEDs to other side of the board, which means they mustbe assembled by hand. Added UART 5 test points.
Parts:
- TP1, TP2: footprint (none) -> TestPoint:TestPoint_Pad_D2.0mm
Changed lines of the file:
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@@
 			)
 		)
-		(property "Footprint" ""
+		(property "Footprint" "TestPoint:TestPoint_Pad_D2.0mm"
 			(at 148.59 128.27 0)
 			(hide yes)
@@
 			)
 		)
-		(property "Footprint" ""
+		(property "Footprint" "TestPoint:TestPoint_Pad_D2.0mm"
 			(at 148.59 133.35 0)
 			(hide yes)

Commit message: Finalize LTELink V2 for production
Parts:
- J5, TP1, TP2: now not fitted
Changed lines of the file:
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@@
 		(on_board yes)
 		(in_pos_files yes)
-		(dnp no)
+		(dnp yes)
 		(fields_autoplaced yes)
 		(property "Reference" "TP1"
@@
 		(on_board yes)
 		(in_pos_files yes)
-		(dnp no)
+		(dnp yes)
 		(property "Reference" "J5"
 			(at 156.21 83.8201 0)
@@
 		(on_board yes)
 		(in_pos_files yes)
-		(dnp no)
+		(dnp yes)
 		(fields_autoplaced yes)
 		(property "Reference" "TP2"
